File: circuit/circuit.kicad_sch (KiCad schematic)
At the start: 77 parts, among them J10 Pedal3_In, J11 Amp_Out, J12 Pedal5_In, J13 Pedal2_In, J14 Pedal4_In, J15 Pedal6_In, J16 Pedal8_In, J17 Pedal7_In, J7 Guitar_In, J9 Pedal1_In, SW1 SW_Push, SW10 SW_Push, SW2 SW_Push, SW3 SW_Push, SW4 SW_Push, SW5 SW_Push, SW6 SW_Push, SW7 SW_Push, SW8 SW_Push, SW9 SW_Push, U1 TL072, U10 74HC595, U10 DG408, U11 DG408, U12 DG408, U2 TL072, U20 ESP32-S3-DevKitC, U3 TL072, U4 DG408, U4 TL072, U5 DG408, U5 TL072, U6 DG408, U7 74HC595, U7 DG408, U8 74HC595, U8 DG408, U9 74HC595, U9 DG408

Commit message: Update circuit.kicad_sch
Swapped DG408 for CD4051B
Parts:
- removed C23: .1uF, symbol Device:C_Small
- removed U10, U11, U12, U4, U5, U6, U7, U8, U9: DG408, DG408DJ-E3:21-0043D_16, symbol DG408:DG408DJ-E3
- added C22: .1uF, symbol Device:C_Small
- added U11, U12, U13, U14, U15, U16, U17, U18, U19: CD4051B, symbol Analog_Switch:CD4051B
Connections:
- net U2_Q1 is gone; now on an unnamed net: U10.14 (SER)
- net +3V3: now also C22.1
- net +5V: now also U11.16 (VDD), U12.16 (VDD), U13.16 (VDD), U14.16 (VDD), U15.16 (VDD), U16.16 (VDD), U17.16 (VDD), U18.16 (VDD), U19.16 (VDD)
- net GND: now also C22.2, U11.4 (X7), U11.6 (INH), U11.8 (VSS), U12.4 (X7), U12.6 (INH), U12.8 (VSS), U13.4 (X7), U13.6 (INH), U13.8 (VSS), U14.4 (X7), U14.6 (INH), U14.8 (VSS), U15.4 (X7), U15.6 (INH), U15.8 (VSS), U16.4 (X7), U16.6 (INH), U16.8 (VSS), U17.4 (X7), U17.6 (INH), U17.8 (VSS), U18.4 (X7), U18.6 (INH), U18.8 (VSS), U19.6 (INH), U19.8 (VSS)
- net Guitar_Out: now also U11.13 (X0), U12.14 (X1), U13.14 (X1), U14.14 (X1), U15.14 (X1), U16.14 (X1), U17.14 (X1), U18.14 (X1)
- net Pedal1_Out: now also U11.14 (X1), U12.13 (X0), U13.15 (X2), U14.15 (X2), U15.15 (X2), U16.15 (X2), U17.15 (X2), U18.15 (X2)
- net Pedal2_Out: now also U11.15 (X2), U12.15 (X2), U13.13 (X0), U14.12 (X3), U15.12 (X3), U16.12 (X3), U17.12 (X3), U18.12 (X3)
- net Pedal3_Out: now also U11.12 (X3), U12.12 (X3), U13.12 (X3), U14.13 (X0), U15.1 (X4), U16.1 (X4), U17.1 (X4), U18.1 (X4)
- net Pedal4_Out: now also U11.1 (X4), U12.1 (X4), U13.1 (X4), U14.1 (X4), U15.13 (X0), U18.5 (X5)
- net Pedal5_Out: now also U11.5 (X5), U16.13 (X0), U18.2 (X6)
- net Pedal6_Out: now also U11.2 (X6), U17.13 (X0)
- net Pedal7_Out: now also U12.5 (X5), U13.5 (X5), U14.5 (X5), U15.5 (X5), U16.5 (X5), U17.5 (X5), U18.13 (X0)
- net Pedal8_Out: now also U12.2 (X6), U13.2 (X6), U14.2 (X6), U15.2 (X6), U16.2 (X6), U17.2 (X6)
- net Row1: now also U11.3 (X), U19.13 (X0)
- net Row2: now also U12.3 (X), U19.14 (X1)
- net Row3: now also U13.3 (X), U19.15 (X2)
- net Row4: now also U14.3 (X), U19.12 (X3)
- net Row5: now also U15.3 (X), U19.1 (X4)
- net Row6: now also U16.3 (X), U19.5 (X5)
- net Row7: now also U17.3 (X), U19.2 (X6)
- net Row8: now also U18.3 (X), U19.4 (X7)
- net U3_Q1: no longer U8.2 (QC)
- net U3_Q2: now also U8.2 (QC); no longer U8.3 (QD)
- net U3_Q3: now also U8.3 (QD); no longer U8.4 (QE)
- net U3_Q4: now also U8.4 (QE); no longer U8.5 (QF)
- net U3_Q5: now also U8.5 (QF); no longer U8.6 (QG)
- net U3_Q6: now also U8.6 (QG); no longer U8.7 (QH)
- net U7_Q0: now also U11.11 (A)
- net U7_Q1: now also U11.10 (B)
- net U7_Q2: now also U11.9 (C)
- net U7_Q3: now also U12.11 (A)
- net U7_Q4: now also U12.10 (B)
- net U7_Q5: now also U12.9 (C)
- net U7_Q6: now also U13.11 (A)
- net U13_Q0 renamed U10_Q0
- net U10_Q0: now also U18.10 (B); no longer U9.15 (QA)
- net U13_Q1 renamed U10_Q1
- net U10_Q1: now also U18.9 (C); no longer U9.1 (QB)
- net U13_Q2 renamed U10_Q2
- net U10_Q2: now also U19.11 (A); no longer U9.2 (QC)
- net U13_Q3 renamed U10_Q3
- net U10_Q3: now also U19.10 (B); no longer U9.3 (QD)
- net U13_Q4 renamed U10_Q4
- net U10_Q4: now also U19.9 (C); no longer U9.4 (QE)
- net U13_Q5: no longer names the net of U10.5 (QF)
- net U13_Q5: no longer U9.5 (QF)
- net U13_Q6: no longer names the net of U10.6 (QG)
- net U13_Q6: no longer U9.6 (QG)
- net U13_Q7: no longer names the net of U10.7 (QH)
- net U13_Q7: no longer U9.7 (QH)
- new net -5V: U11.7 (VEE), U12.7 (VEE), U13.7 (VEE), U14.7 (VEE), U15.7 (VEE), U16.7 (VEE), U17.7 (VEE), U18.7 (VEE), U19.7 (VEE)
- new net Matrix_out: U19.3 (X)
- new net U3_Q7: U8.7 (QH)
- new net U8_Q0: U13.10 (B)
- new net U8_Q1: U13.9 (C)
- new net U8_Q2: U14.11 (A)
- new net U8_Q3: U14.10 (B)
- new net U8_Q4: U14.9 (C)
- new net U8_Q5: U15.11 (A)
- new net U8_Q6: U15.10 (B)
- new net U9_Q0: U15.9 (C), U9.15 (QA)
- new net U9_Q1: U16.11 (A), U9.1 (QB)
- new net U9_Q2: U16.10 (B), U9.2 (QC)
- new net U9_Q3: U16.9 (C), U9.3 (QD)
- new net U9_Q4: U17.11 (A), U9.4 (QE)
- new net U9_Q5: U17.10 (B), U9.5 (QF)
- new net U9_Q6: U17.9 (C), U9.6 (QG)
- new net U9_Q7: U18.11 (A), U9.7 (QH)
- no-connect marks 2 -> 4
Other:
- note added: "Guitar Routing"
- note added: "Output Selector"
- note added: "Pedal 1 Routing"
- note added: "Pedal 2 Routing"
- note added: "Pedal 3 Routing"
- note added: "Pedal 4 Routing"
- note added: "Pedal 5 Routing"
- note added: "Pedal 6 Routing"
- note added: "Pedal 7 Routing"

Commit message: Update circuit.kicad_sch
Added Power supplies and Nets.
Parts:
- removed C28, C29: 10uF, symbol Device:C_Small
- added C23, C25, C26, C30, C32: 0.1mF, symbol Device:C_Small
- added C24: 100mF, symbol Device:C_Small
- added C27, C31: 0.33mF, symbol Device:C_Small
- added C33, C34: 10mF, symbol Device:C_Polarized_Small
- added D1: 1N4007, Diode_THT:D_DO-41_SOD81_P10.16mm_Horizontal, symbol Diode:1N4007
- added F1: Polyfuse_Small, symbol Device:Polyfuse_Small
- added J1: Barrel_Jack, symbol Connector:Barrel_Jack
- added U21: LM7805_TO220, Package_TO_SOT_THT:TO-220-3_Vertical, symbol Regulator_Linear:LM7805_TO220
- added U22: LM7905_TO220, Package_TO_SOT_THT:TO-220-3_Vertical, symbol Regulator_Linear:LM7905_TO220
- added U23: AMS1117-3.3, Package_TO_SOT_SMD:SOT-223-3_TabPin2, symbol Regulator_Linear:AMS1117-3.3
- added U6: TMA-1215D, Converter_DCDC:Converter_DCDC_TRACO_TMA-05xxD_12xxD_Dual_THT, symbol Converter_DCDC:TMA-1215D
Connections:
- net +5V: now also C30.1
- net -5V: now also C32.1
- net GND: now also C23.1, C24.1, C25.2, C26.2, J1.1, U21.2 (GND), U22.1 (GND), U23.1 (GND), U6.2 (-Vin)
- net +3V3 renamed 3.3V
- net 3.3V: now also C34.2; no longer C17.1, U7.10 (~{SRCLR}), U7.16 (VCC)
- net +9V renamed +15V
- net +15V: now also C26.1, U6.6 (+Vout)
- net -9V renamed -15V
- net -15V: now also C25.1, U6.4 (-Vout)
- new net: C31.1, U22.2 (VI)
- new net: C34.1, U23.2 (VO)
- new net: C33.2, U23.3 (VI)
- new net: C27.1, U21.1 (VI)
- new net: D1.1 (K), F1.2
- new net: C17.1, U7.10 (~{SRCLR}), U7.16 (VCC)
- new net: C30.2, U21.3 (VO)
- new net: D1.2 (A), J1.2
- new net: C32.2, U22.3 (VO)
- new net VIN_12V: C23.2, C24.2, C27.2, C31.2, C33.1, F1.1, U6.1 (+Vin)

Commit message: Update circuit.kicad_sch
Parts:
- removed C21: C_Small, symbol Device:C_Small
- removed R1: R_Small, symbol Device:R_Small
- added C28, C29, C35, C36, C37, C38, C39, C40, C41, C42: 0.1mF, symbol Device:C_Small
Connections:
- net GND: now also SW1.2, SW10.2, SW2.2, SW3.2, SW4.2, SW5.2, SW6.2, SW7.2, SW8.2, SW9.2, C28.1, C29.1, C35.1, C36.1, C37.1, C38.1, C39.1, C40.1, C41.1, C42.1
- net at SW3.1, U20.12 (GPIO8/ADC1_CH7): now also C40.2
- net at SW6.1, U20.17 (GPIO11/ADC2_CH0): now also C37.2
- net at SW5.1, U20.16 (GPIO10/ADC1_CH9): now also C38.2
- net at SW9.1, U20.20 (GPIO14/ADC2_CH3): now also C29.2
- net at SW2.1, U20.7 (GPIO7/ADC1_CH6): now also C41.2
- net at SW8.1, U20.19 (GPIO13/ADC2_CH2): now also C35.2
- net at SW10.1, U20.8 (GPIO15/ADC2_CH4/32K_P): now also C28.2
- net at SW4.1, U20.15 (GPIO9/ADC1_CH8): now also C39.2
- net at SW1.1, U20.6 (GPIO6/ADC1_CH5): now also C42.2
- net at SW7.1, U20.18 (GPIO12/ADC2_CH1): now also C36.2
- no-connect marks 4 -> 25
Other:
- moved on the sheet: SW1, SW10, SW2, SW3, SW4, SW5, SW6, SW7, SW8, SW9

Commit message: Update circuit.kicad_sch
Parts:
- renumbered C17 to C47, C18 to C48, C19 to C49
Connections:
- net Matrix_out is gone; now on net Matrix_Out: U19.3 (X)
- net SR_0E is gone; now on net SR_OE: U20.25 (GPIO19/USB_D-)
- net U3_Q0 is gone; now on net U8_Q0: U8.15 (QA)
- net U3_Q1 is gone; now on net U8_Q1: U8.1 (QB)
- net U3_Q2 is gone; now on net U8_Q2: U8.2 (QC)
- net U3_Q3 is gone; now on net U8_Q3: U8.3 (QD)
- net U3_Q4 is gone; now on net U8_Q4: U8.4 (QE)
- net U3_Q5 is gone; now on net U8_Q5: U8.5 (QF)
- net U3_Q6 is gone; now on net U8_Q6: U8.6 (QG)
- net 3.3V: now also C47.1, U7.10 (~{SRCLR}), U7.16 (VCC)
- net U10_Q0: now also U19.11 (A); no longer U18.10 (B)
- net U10_Q1: now also U19.10 (B); no longer U18.9 (C)
- net U10_Q2: now also U19.9 (C); no longer U19.11 (A)
- net U7_Q7: now also U13.10 (B)
- net U8_Q0: now also U13.9 (C); no longer U13.10 (B)
- net U8_Q1: now also U14.11 (A); no longer U13.9 (C)
- net U8_Q2: now also U14.10 (B); no longer U14.11 (A)
- net U8_Q3: now also U14.9 (C); no longer U14.10 (B)
- net U8_Q4: now also U15.11 (A); no longer U14.9 (C)
- net U8_Q5: now also U15.10 (B); no longer U15.11 (A)
- net U8_Q6: now also U15.9 (C); no longer U15.10 (B)
- net U9_Q0: now also U16.10 (B); no longer U15.9 (C)
- net U9_Q1: now also U16.9 (C); no longer U16.11 (A)
- net U9_Q2: now also U17.11 (A); no longer U16.10 (B)
- net U9_Q3: now also U17.10 (B); no longer U16.9 (C)
- net U9_Q4: now also U17.9 (C); no longer U17.11 (A)
- net U9_Q5: now also U18.11 (A); no longer U17.10 (B)
- net U9_Q6: now also U18.10 (B); no longer U17.9 (C)
- net U9_Q7: now also U18.9 (C); no longer U18.11 (A)
- net Amp_Out renamed Matrix_Out
- net U10_Q3: no longer names the net of U10.3 (QD)
- net U10_Q3: no longer U19.10 (B)
- net U10_Q4: no longer names the net of U10.4 (QE)
- net U10_Q4: no longer U19.9 (C)
- net U3_Q7 renamed U8_Q7
- net U8_Q7: now also U16.11 (A)
- no-connect marks 25 -> 28

Commit message: Circuit nearly complete. Need more decoupling Caps.
Connections:
- net 3.3V: now also C28.1, C29.1, C35.1, C36.1, C37.1, C38.1, C39.1, C40.1, C41.1, C42.1, SW1.2, SW10.2, SW2.2, SW3.2, SW4.2, SW5.2, SW6.2, SW7.2, SW8.2, SW9.2
- net GND: no longer C28.1, C29.1, C35.1, C36.1, C37.1, C38.1, C39.1, C40.1, C41.1, C42.1, SW1.2, SW10.2, SW2.2, SW3.2, SW4.2, SW5.2, SW6.2, SW7.2, SW8.2, SW9.2
Other:
- moved on the sheet: C27, C31, C33

Commit message: Continued prgress on circuit. Split digital and analog gnd.
Parts:
- added NT1: NetTie_2, NetTie:NetTie-2_THT_Pad1.0mm, symbol Device:NetTie_2
- C1, C10, C11, C12, C13, C14, C15, C16, C17, C18, C19, C2, C20, C22, C23, C24, C25, C26, C27, C28, C29, C3, C30, C31, C32, C33, C34, C35, C36, C37, C38, C39, C4, C40, C41, C42, C47, C48, C49, C5, C6, C7, C8, C9: footprint (none) -> Capacitor_THT:C_Axial_L3.8mm_D2.6mm_P7.50mm_Horizontal
- Disp1: footprint (none) -> Connector_Wire:SolderWire-1.5sqmm_1x04_P6mm_D1.7mm_OD3mm
- F1: footprint (none) -> TerminalBlock_Phoenix:TerminalBlock_Phoenix_PTSM-0,5-2-2.5-H-THR_1x02_P2.50mm_Horizontal
- J1: footprint (none) -> Connector_BarrelJack:BarrelJack_CUI_PJ-063AH_Horizontal_CircularHoles
- J10, J11, J12, J13, J14, J15, J16, J17, J7, J9, SW1, SW10, SW2, SW3, SW4, SW5, SW6, SW7, SW8, SW9: footprint (none) -> Connector_Wire:SolderWire-0.1sqmm_1x02_P3.6mm_D0.4mm_OD1mm
- R10, R2, R3, R4, R5, R6, R7, R8, R9: footprint (none) -> Resistor_THT:R_Axial_DIN0204_L3.6mm_D1.6mm_P5.08mm_Horizontal
- U1, U2, U3, U4, U5: footprint (none) -> Package_DIP:CERDIP-8_W7.62mm_SideBrazed
- U10, U11, U12, U13, U14, U15, U16, U17, U18, U19, U7, U8, U9: footprint (none) -> Package_DIP:CERDIP-16_W7.62mm_SideBrazed
- U20: footprint PCM_Espressif:ESP32-S3-DevKitC -> Esp32 DevKits:ESP32-S3-DevKitC
Connections:
- net 3.3V: no longer C28.1, C29.1, C35.1, C36.1, C37.1, C38.1, C39.1, C40.1, C41.1, C42.1, SW1.2, SW10.2, SW2.2, SW3.2, SW4.2, SW5.2, SW6.2, SW7.2, SW8.2, SW9.2
- net GND: now also C28.1, C29.1, C35.1, C36.1, C37.1, C38.1, C39.1, C40.1, C41.1, C42.1, SW1.2, SW10.2, SW2.2, SW3.2, SW4.2, SW5.2, SW6.2, SW7.2, SW8.2, SW9.2, NT1.1; no longer C11.2, C12.1, C13.2, C14.1, C15.2, C16.1, C17.2, C18.1, C19.2, C20.1, C25.2, C26.2, J10.S, J11.S, J12.S, J13.S, J14.S, J15.S, J16.S, J17.S, J7.S, J9.S, U11.4 (X7), U11.6 (INH), U11.8 (VSS), U12.4 (X7), U12.6 (INH), U12.8 (VSS), U13.4 (X7), U13.6 (INH), U13.8 (VSS), U14.4 (X7), U14.6 (INH), U14.8 (VSS), U15.4 (X7), U15.6 (INH), U15.8 (VSS), U16.4 (X7), U16.6 (INH), U16.8 (VSS), U17.4 (X7), U17.6 (INH), U17.8 (VSS), U18.4 (X7), U18.6 (INH), U18.8 (VSS), U19.6 (INH), U19.8 (VSS), U6.2 (-Vin)
- new net AGND: C11.2, C12.1, C13.2, C14.1, C15.2, C16.1, C17.2, C18.1, C19.2, C20.1, C25.2, C26.2, J10.S, J11.S, J12.S, J13.S, J14.S, J15.S, J16.S, J17.S, J7.S, J9.S, NT1.2, U11.4 (X7), U11.6 (INH), U11.8 (VSS), U12.4 (X7), U12.6 (INH), U12.8 (VSS), U13.4 (X7), U13.6 (INH), U13.8 (VSS), U14.4 (X7), U14.6 (INH), U14.8 (VSS), U15.4 (X7), U15.6 (INH), U15.8 (VSS), U16.4 (X7), U16.6 (INH), U16.8 (VSS), U17.4 (X7), U17.6 (INH), U17.8 (VSS), U18.4 (X7), U18.6 (INH), U18.8 (VSS), U19.6 (INH), U19.8 (VSS), U6.2 (-Vin)

Commit message: Editing Circuit for readability.
Parts:
- removed C1, C10, C2, C3, C4, C5, C6, C7, C8, C9: 1mF, Capacitor_THT:C_Axial_L3.8mm_D2.6mm_P7.50mm_Horizontal, symbol Device:C_Small
- removed C11, C12, C13, C14, C15, C16, C17, C18, C19, C20: 0.1uF, Capacitor_THT:C_Axial_L3.8mm_D2.6mm_P7.50mm_Horizontal, symbol Device:C_Small
- removed C22, C47, C48, C49: .1uF, Capacitor_THT:C_Axial_L3.8mm_D2.6mm_P7.50mm_Horizontal, symbol Device:C_Small
- removed C23, C25, C26, C30, C32: 0.1mF, Capacitor_THT:C_Axial_L3.8mm_D2.6mm_P7.50mm_Horizontal, symbol Device:C_Small
- removed C24: 100mF, Capacitor_THT:C_Axial_L3.8mm_D2.6mm_P7.50mm_Horizontal, symbol Device:C_Small
- removed C27, C31: 0.33mF, Capacitor_THT:C_Axial_L3.8mm_D2.6mm_P7.50mm_Horizontal, symbol Device:C_Small
- removed C33, C34: 10mF, Capacitor_THT:C_Axial_L3.8mm_D2.6mm_P7.50mm_Horizontal, symbol Device:C_Polarized_Small
- removed D1: 1N4007, Diode_THT:D_DO-41_SOD81_P10.16mm_Horizontal, symbol Diode:1N4007
- removed F1: Polyfuse_Small, TerminalBlock_Phoenix:TerminalBlock_Phoenix_PTSM-0,5-2-2.5-H-THR_1x02_P2.50mm_Horizontal, symbol Device:Polyfuse_Small
- removed J1: Barrel_Jack, Connector_BarrelJack:BarrelJack_CUI_PJ-063AH_Horizontal_CircularHoles, symbol Connector:Barrel_Jack
- removed J10: Pedal3_In, Connector_Wire:SolderWire-0.1sqmm_1x02_P3.6mm_D0.4mm_OD1mm, symbol Connector_Audio:AudioJack2
- removed J11: Amp_Out, Connector_Wire:SolderWire-0.1sqmm_1x02_P3.6mm_D0.4mm_OD1mm, symbol Connector_Audio:AudioJack2
- removed J12: Pedal5_In, Connector_Wire:SolderWire-0.1sqmm_1x02_P3.6mm_D0.4mm_OD1mm, symbol Connector_Audio:AudioJack2
- removed J13: Pedal2_In, Connector_Wire:SolderWire-0.1sqmm_1x02_P3.6mm_D0.4mm_OD1mm, symbol Connector_Audio:AudioJack2
- removed J14: Pedal4_In, Connector_Wire:SolderWire-0.1sqmm_1x02_P3.6mm_D0.4mm_OD1mm, symbol Connector_Audio:AudioJack2
- removed J15: Pedal6_In, Connector_Wire:SolderWire-0.1sqmm_1x02_P3.6mm_D0.4mm_OD1mm, symbol Connector_Audio:AudioJack2
- removed J16: Pedal8_In, Connector_Wire:SolderWire-0.1sqmm_1x02_P3.6mm_D0.4mm_OD1mm, symbol Connector_Audio:AudioJack2
- removed J17: Pedal7_In, Connector_Wire:SolderWire-0.1sqmm_1x02_P3.6mm_D0.4mm_OD1mm, symbol Connector_Audio:AudioJack2
- removed J7: Guitar_In, Connector_Wire:SolderWire-0.1sqmm_1x02_P3.6mm_D0.4mm_OD1mm, symbol Connector_Audio:AudioJack2
- removed J9: Pedal1_In, Connector_Wire:SolderWire-0.1sqmm_1x02_P3.6mm_D0.4mm_OD1mm, symbol Connector_Audio:AudioJack2
- removed R10, R2, R3, R4, R5, R6, R7, R8, R9: 10k, Resistor_THT:R_Axial_DIN0204_L3.6mm_D1.6mm_P5.08mm_Horizontal, symbol Device:R_US
- removed U1, U2, U3, U4, U5: TL072, Package_DIP:CERDIP-8_W7.62mm_SideBrazed, symbol Bay:TL072
- removed U10, U7, U8, U9: 74HC595, Package_DIP:CERDIP-16_W7.62mm_SideBrazed, symbol 74xx:74HC595
- removed U11, U12, U13, U14, U15, U16, U17, U18, U19: CD4051B, Package_DIP:CERDIP-16_W7.62mm_SideBrazed, symbol Analog_Switch:CD4051B
- removed U21: LM7805_TO220, Package_TO_SOT_THT:TO-220-3_Vertical, symbol Regulator_Linear:LM7805_TO220
- removed U22: LM7905_TO220, Package_TO_SOT_THT:TO-220-3_Vertical, symbol Regulator_Linear:LM7905_TO220
- removed U23: AMS1117-3.3, Package_TO_SOT_SMD:SOT-223-3_TabPin2, symbol Regulator_Linear:AMS1117-3.3
- removed U6: TMA-1215D, Converter_DCDC:Converter_DCDC_TRACO_TMA-05xxD_12xxD_Dual_THT, symbol Converter_DCDC:TMA-1215D
- renumbered C42 to C103, C41 to C107, C40 to C109, C39 to C112, C38 to C113, C37 to C114, C36 to C117, C35 to C120, C29 to C123, C28 to C126, Disp1 to Disp101, NT1 to NT101, SW1 to SW101, SW2 to SW102, SW3 to SW103, SW4 to SW104, SW5 to SW105, SW6 to SW106, SW7 to SW107, SW8 to SW108, SW9 to SW109, SW10 to SW110, U20 to U103
Connections:
- no-connect marks 28 -> 21
Other:
- added sheet Buffers (Buffers.kicad_sch)
- added sheet IO Routing (iorouting.kicad_sch)
- added sheet Pedal Routing 1 - 4 (pedal_routing_1-4.kicad_sch)
- added sheet Pedal Routing 5 - 8 (pedal_routing_4-8.kicad_sch)
- added sheet Power (Power.kicad_sch)
- added sheet Shift Registers (shift_registers.kicad_sch)
- note removed: "Guitar Routing"
- note removed: "Output Selector"
- note removed: "Pedal 1 Routing"
- note removed: "Pedal 2 Routing"
- note removed: "Pedal 3 Routing"
- note removed: "Pedal 4 Routing"
- note removed: "Pedal 5 Routing"
- note removed: "Pedal 6 Routing"
- note removed: "Pedal 7 Routing"
- moved on the sheet: NT101

Commit message: Rebuilt bus and matrix.
Parts:
- renumbered C103 to C101, C107 to C102, C109 to C103, C112 to C104, C113 to C105, C114 to C106, C117 to C107, C120 to C108, C123 to C109, C126 to C110, U103 to U5
Other:
- sheet IO Routing ports: added U10_Q[0..5], U7_Q[0..7]; removed none
- sheet Pedal Routing 1 - 4 ports: added U7_Q[0..7], U8_Q[0..7]; removed none
- sheet Pedal Routing 5 - 8 ports: added U10_Q[0..5], U8_Q[0..7], U9_Q[0..7]; removed none
- sheet Shift Registers ports: added U10_Q[0..5], U7_Q[0..7], U8_Q[0..7], U9_Q[0..7]; removed none
