File: circuit/circuit.kicad_sch (KiCad schematic)
At the start: 27 parts, among them SW101 Pedal_1, SW102 Pedal_2, SW103 Pedal_3, SW104 Pedal_4, SW105 Pedal_5, SW106 Pedal_6, SW107 Pedal_7, SW108 Pedal_8, SW109 Program, SW110 Preset, U101 ESP32-S3-DevKitC

Commit message: Labels for headers on PCB
Parts:
- C101, C110: footprint Capacitor_THT:C_Disc_D3.0mm_W2.0mm_P2.50mm -> Capacitor_THT:C_Disc_D5.0mm_W2.5mm_P2.50mm
- C102: renamed from C106; footprint Capacitor_THT:C_Disc_D3.0mm_W2.0mm_P2.50mm -> Capacitor_THT:C_Disc_D5.0mm_W2.5mm_P2.50mm
- C103: renamed from C102; footprint Capacitor_THT:C_Disc_D3.0mm_W2.0mm_P2.50mm -> Capacitor_THT:C_Disc_D5.0mm_W2.5mm_P2.50mm
- C104: renamed from C107; footprint Capacitor_THT:C_Disc_D3.0mm_W2.0mm_P2.50mm -> Capacitor_THT:C_Disc_D5.0mm_W2.5mm_P2.50mm
- C105: renamed from C103; footprint Capacitor_THT:C_Disc_D3.0mm_W2.0mm_P2.50mm -> Capacitor_THT:C_Disc_D5.0mm_W2.5mm_P2.50mm
- C106: renamed from C108; footprint Capacitor_THT:C_Disc_D3.0mm_W2.0mm_P2.50mm -> Capacitor_THT:C_Disc_D5.0mm_W2.5mm_P2.50mm
- C107: renamed from C104; footprint Capacitor_THT:C_Disc_D3.0mm_W2.0mm_P2.50mm -> Capacitor_THT:C_Disc_D5.0mm_W2.5mm_P2.50mm
- C108: renamed from C109; footprint Capacitor_THT:C_Disc_D3.0mm_W2.0mm_P2.50mm -> Capacitor_THT:C_Disc_D5.0mm_W2.5mm_P2.50mm
- C109: renamed from C105; footprint Capacitor_THT:C_Disc_D3.0mm_W2.0mm_P2.50mm -> Capacitor_THT:C_Disc_D5.0mm_W2.5mm_P2.50mm
- renumbered SW106 to SW102, SW102 to SW103, SW107 to SW104, SW103 to SW105, SW108 to SW106, SW104 to SW107, SW109 to SW108, SW105 to SW109
Other:
- sheet IO Routing ports: added U701_Q[0..7]; removed U7_Q[0..7]
- sheet Matrix Shift Registers ports: added U701_Q[0..7], U702_Q[0..7], U703_Q[0..7], U704_Q[0..3]; removed U10_Q[0..3], U7_Q[0..7], U8_Q[0..7], U9_Q[0..7]
- sheet Pedal Routing 1 - 4 ports: added U701_Q[0..7], U702_Q[0..7]; removed U7_Q[0..7], U8_Q[0..7]
- sheet Pedal Routing 5 - 8 ports: added U703_Q[0..7], U704_Q[0..3]; removed U10_Q[0..3], U9_Q[0..7]
