File: circuit/iorouting.kicad_sch (KiCad schematic)
At the start: 2 parts, among them U109 CD4051B, U119 CD4051B

Commit message: Rebuilt bus and matrix.
Parts:
- renumbered U109 to U15, U119 to U25
Connections:
- net Row2 is gone; now on net ROW_2: U25.14 (X1)
- net Row3 is gone; now on net ROW_3: U25.15 (X2)
- net Row4 is gone; now on net ROW_4: U25.12 (X3)
- net Row5 is gone; now on net ROW_5: U25.1 (X4)
- net Row6 is gone; now on net ROW_6: U25.5 (X5)
- net Row7 is gone; now on net ROW_7: U25.2 (X6)
- net AGND: no longer U15.4 (X7)
- net Guitar_Out renamed ROW_1
- net ROW_1: now also U25.13 (X0)
- net Matrix_Out renamed MATRIX_OUT
- net Pedal1_Out renamed ROW_2
- net Pedal2_Out renamed ROW_3
- net Pedal3_Out renamed ROW_4
- net Pedal4_Out renamed ROW_5
- net Pedal5_Out renamed ROW_6
- net Pedal6_Out renamed ROW_7
- net Row1 renamed GUITAR_IN
- net GUITAR_IN: no longer U25.13 (X0)
- net Row8 renamed ROW_8
- net ROW_8: now also U15.4 (X7)
- net U10_Q0 renamed U10_Q3
- net U10_Q1 renamed U10_Q4
- net U10_Q2 renamed U10_Q5

Commit message: Hopefully close to finished
Parts:
- added C111, C112, C113, C114, C115, C116: 0.1mF, Capacitor_THT:C_Axial_L3.8mm_D2.6mm_P7.50mm_Horizontal, symbol Device:C_Small
- added U101: ADG419BN, Package_DIP:DIP-8_W7.62mm, symbol Analog_Switch:ADG419BN
- renumbered U15 to U16, U25 to U20
Connections:
- net +5V: now also C112.1, C114.2, C116.2, U101.5 (VL)
- net -5V: now also C113.1, C115.1
- net AGND: now also C111.2, C112.2, C113.2, C114.1, C115.2, C116.1, U101.3 (GND)
- net U7_Q0: now also U101.6; no longer U16.11 (A)
- net U7_Q2: now also U16.11 (A); no longer U16.9 (C)
- net MATRIX_OUT: no longer names the net of U20.3 (X)
- net MATRIX_OUT: now also U101.2
- net U10_Q3 renamed U7_Q5
- net U10_Q4 renamed U7_Q6
- net U10_Q5 renamed U7_Q7
- net U7_Q1 renamed U7_Q3
- new net +15V: C111.1, U101.4 (V+)
- new net -15V: U101.7 (V-)
- new net MATRIX_OUT_PRE: U101.1
- new net ROW_9: U101.8
- new net U7_Q4: U16.9 (C)
Other:
- note added: "Output Mux 1"
- note removed: "Output Selector"
