File: circuit/shift_registers.kicad_sch (KiCad schematic)
At the start: 8 parts, among them U107 74HC595, U108 74HC595, U111 74HC595, U112 74HC595

Commit message: Rebuilt bus and matrix.
Parts:
- renumbered C131 to C701, C132 to C702, C133 to C703, C134 to C704, U112 to U10, U107 to U7, U108 to U8, U111 to U9
Connections:
- net U10_Q3: now reaches U10.3 (QD)
- net U10_Q4: now reaches U10.4 (QE)
- net U10_Q5: now reaches U10.5 (QF)
- no-connect marks 6 -> 3

Commit message: Hopefully close to finished
Connections:
- net U10_Q6: now reaches U10.6 (QG)
- net U10_Q7: now reaches U10.7 (QH)
- net U7_Q1: no longer names the net of U7.1 (QB)
- no-connect marks 3 -> 2
Changed lines of the file:
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@@
-	)
-	(no_connect
-		(at 204.47 139.7)
-	)
-	(no_connect
-		(at 204.47 142.24)
 	)
 	(no_connect
 		(at 204.47 147.32)
 	)
+	(no_connect
+		(at 133.35 72.39)
+	)
 	(bus_entry
 		(at 142.24 82.55)
@@
 	)
 	(bus_entry
-		(at 144.78 69.85)
+		(at 218.44 137.16)
 		(size -2.54 2.54)
 		(stroke
@@
 	(bus_entry
 		(at 147.32 121.92)
+		(size -2.54 2.54)
+		(stroke
+			(width 0)
+			(type default)
+		)
+	)
+	(bus_entry
+		(at 218.44 139.7)
 		(size -2.54 2.54)
 		(stroke
@@
 	)
 	(bus_entry
-		(at 142.24 72.39)
-		(size 2.54 -2.54)
-		(stroke
-			(width 0)
-			(type default)
-		)
-	)
-	(bus_entry
 		(at 147.32 132.08)
 		(size -2.54 2.54)
@@
 	(bus
 		(pts
-			(xy 144.78 69.85) (xy 144.78 72.39)
+			(xy 144.78 68.58) (xy 144.78 72.39)
 		)
 		(stroke
@@
 		)
 	)
+	(wire
+		(pts
+			(xy 204.47 142.24) (xy 215.9 142.24)
+		)
+		(stroke
+			(width 0)
+			(type default)
+		)
+	)
 	(bus
 		(pts
@@
 		)
 	)
+	(bus
+		(pts
+			(xy 218.44 137.16) (xy 218.44 139.7)
+		)
+		(stroke
+			(width 0)
+			(type default)
+		)
+	)
 	(wire
 		(pts
@@
 		)
 	)
-	(wire
-		(pts
-			(xy 133.35 72.39) (xy 142.24 72.39)
-		)
-		(stroke
-			(width 0)
-			(type default)
-		)
-	)
 	(bus
 		(pts
@@
 	(bus
 		(pts
+			(xy 218.44 134.62) (xy 218.44 137.16)
+		)
+		(stroke
+			(width 0)
+			(type default)
+		)
+	)
+	(bus
+		(pts
 			(xy 147.32 129.54) (xy 147.32 127)
 		)
@@
 	(bus
 		(pts
-			(xy 144.78 68.58) (xy 144.78 69.85)
-		)
-		(stroke
-			(width 0)
-			(type default)
-		)
-	)
-	(bus
-		(pts
 			(xy 203.2 72.39) (xy 203.2 69.85)
 		)
@@
 		(pts
 			(xy 218.44 129.54) (xy 218.44 132.08)
+		)
+		(stroke
+			(width 0)
+			(type default)
+		)
+	)
+	(wire
+		(pts
+			(xy 204.47 139.7) (xy 215.9 139.7)
 		)
 		(stroke
@@
 		)
 	)
-	(label "U7_Q1"
-		(at 135.89 72.39 0)
-		(effects
-			(font
-				(size 1.27 1.27)
-			)
-			(justify left bottom)
-		)
-	)
 	(label "U8_Q2"
 		(at 194.31 74.93 0)
@@
 		)
 	)
+	(label "U10_Q6"
+		(at 204.47 139.7 0)
+		(effects
+			(font
+				(size 1.27 1.27)
+			)
+			(justify left bottom)
+		)
+	)
 	(label "U8_Q1"
 		(at 194.31 72.39 0)
@@
 		)
 	)
+	(label "U10_Q7"
+		(at 204.47 142.24 0)
+		(effects
+			(font
+				(size 1.27 1.27)
+			)
+			(justify left bottom)
+		)
+	)
 	(label "U9_Q4"
 		(at 133.35 132.08 0)
@@
 		)
 	)
-	(label "U10_Q[0..5]"
+	(label "U10_Q[0..7]"
 		(at 223.52 119.38 0)
 		(effects
@@
 		)
 	)
-	(hierarchical_label "U10_Q[0..5]"
+	(hierarchical_label "U10_Q[0..7]"
 		(shape output)
 		(at 222.25 120.65 0)

Commit message: Created pdf and made minor readabilty changes.
Other:
- title: (none) -> ESP332 Guitar Patch Bay
Changed lines of the file:
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@@
 	(generator "eeschema")
 	(generator_version "9.0")
-	(paper "A4")
+	(paper "USLetter")
+	(title_block
+		(title "ESP332 Guitar Patch Bay")
+		(date "2025-05-27")
+		(rev "1")
+	)
 	(junction
 		(at 203.2 64.77)

Commit message: Added LEDs and shift registers
Connections:
- net SR_DS renamed MATRIX_SR_DS
Changed lines of the file:
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@@
 	(wire
 		(pts
-			(xy 104.14 69.85) (xy 113.03 69.85)
+			(xy 110.49 69.85) (xy 113.03 69.85)
 		)
 		(stroke
@@
 		)
 	)
-	(global_label "SR_DS"
-		(shape input)
-		(at 104.14 69.85 180)
-		(fields_autoplaced yes)
-		(effects
-			(font
-				(size 1.27 1.27)
-			)
-			(justify right)
-		)
-		(property "Intersheetrefs" "${INTERSHEET_REFS}"
-			(at 95.2282 69.85 0)
-			(effects
-				(font
+	(global_label "MATRIX_SR_DS"
+		(shape input)
+		(at 110.49 69.85 180)
+		(fields_autoplaced yes)
+		(effects
+			(font
+				(size 1.27 1.27)
+			)
+			(justify right)
+		)
+		(property "Intersheetrefs" "${INTERSHEET_REFS}"
+			(at 101.5782 69.85 0)
+			(effects
+				(font

Commit message: Very tentative PCB layout, Code compiles but needs major functionality testing.
Parts:
- C701, C702, C703, C704: value .1uF -> 0.1uF
Changed lines of the file:
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@@
 			)
 		)
-		(property "Value" ".1uF"
+		(property "Value" "0.1uF"
 			(at 179.07 151.1362 0)
 			(effects
@@
 			)
 		)
-		(property "Value" ".1uF"
+		(property "Value" "0.1uF"
 			(at 107.95 148.5962 0)
 			(effects
@@
 			)
 		)
-		(property "Value" ".1uF"
+		(property "Value" "0.1uF"
 			(at 107.95 96.5262 0)
 			(effects
@@
 			)
 		)
-		(property "Value" ".1uF"
+		(property "Value" "0.1uF"
 			(at 167.64 100.3362 0)
 			(effects

Commit message: Rebuilt Matrix and added inhibit function.
Matrix was flawed, It now supports 8 FX loops (pedals) in any order. Or optionally none at all with a buffered bypass, or anywhere in between. The inhibit function will allow the option to press any loop foot switch an enable or disable it without reprogramming.
Connections:
- net U7_Q1: now reaches U7.1 (QB)
- net U10_Q4: no longer names the net of U10.4 (QE)
- net U10_Q5: no longer names the net of U10.5 (QF)
- net U10_Q6: no longer names the net of U10.6 (QG)
- net U10_Q7: no longer names the net of U10.7 (QH)
- no-connect marks 2 -> 5
Other:
- moved on the sheet: C701, C702, C703, C704, U10, U7, U8, U9

Commit message: Re-annotation of circuit, new PCB routing, updated PDF
Parts:
- renumbered U7 to U701, U8 to U702, U9 to U703, U10 to U704
Changed lines of the file:
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@@
 		(dnp no)
 		(fields_autoplaced yes)
-		(property "Reference" "U9"
+		(property "Reference" "U703"
 			(at 73.2633 78.74 0)
 			(effects
@@
 			(project "circuit"
 				(path "/420e3d7a-6c9a-4806-b4be-05d56aeb21de/4760116a-7aa4-465f-87dd-a53dbe30c185"
-					(reference "U9")
+					(reference "U703")
 					(unit 1)
 				)
@@
 		(dnp no)
 		(fields_autoplaced yes)
-		(property "Reference" "U7"
+		(property "Reference" "U701"
 			(at 73.2633 26.2 0)
 			(effects
@@
 			(project "circuit"
 				(path "/420e3d7a-6c9a-4806-b4be-05d56aeb21de/4760116a-7aa4-465f-87dd-a53dbe30c185"
-					(reference "U7")
+					(reference "U701")
 					(unit 1)
 				)
@@
 		(dnp no)
 		(fields_autoplaced yes)
-		(property "Reference" "U10"
+		(property "Reference" "U704"
 			(at 144.3833 81.28 0)
 			(effects
@@
 			(project "circuit"
 				(path "/420e3d7a-6c9a-4806-b4be-05d56aeb21de/4760116a-7aa4-465f-87dd-a53dbe30c185"
-					(reference "U10")
+					(reference "U704")
 					(unit 1)
 				)
@@
 		(dnp no)
 		(fields_autoplaced yes)
-		(property "Reference" "U8"
+		(property "Reference" "U702"
 			(at 132.9533 26.2 0)
 			(effects
@@
 			(project "circuit"
 				(path "/420e3d7a-6c9a-4806-b4be-05d56aeb21de/4760116a-7aa4-465f-87dd-a53dbe30c185"
-					(reference "U8")
-					(unit 1)
-				)
+					(reference "U702")
+					(unit 1)
+				)

Commit message: Added ferrite beads and tweaked PCB
Parts:
- C701, C702, C703, C704: footprint Capacitor_THT:C_Axial_L3.8mm_D2.6mm_P7.50mm_Horizontal -> Capacitor_THT:C_Disc_D3.0mm_W2.0mm_P2.50mm
- U701, U702, U703, U704: footprint Package_DIP:CERDIP-16_W7.62mm_SideBrazed -> Package_DIP:DIP-16_W7.62mm
Changed lines of the file:
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@@
 			)
 		)
-		(property "Footprint" "Capacitor_THT:C_Axial_L3.8mm_D2.6mm_P7.50mm_Horizontal"
+		(property "Footprint" "Capacitor_THT:C_Disc_D3.0mm_W2.0mm_P2.50mm"
 			(at 124.46 114.3 0)
 			(effects
@@
 			)
 		)
-		(property "Footprint" "Package_DIP:CERDIP-16_W7.62mm_SideBrazed"
+		(property "Footprint" "Package_DIP:DIP-16_W7.62mm"
 			(at 71.12 96.52 0)
 			(effects
@@
 			)
 		)
-		(property "Footprint" "Capacitor_THT:C_Axial_L3.8mm_D2.6mm_P7.50mm_Horizontal"
+		(property "Footprint" "Capacitor_THT:C_Disc_D3.0mm_W2.0mm_P2.50mm"
 			(at 53.34 111.76 0)
 			(effects
@@
 			)
 		)
-		(property "Footprint" "Package_DIP:CERDIP-16_W7.62mm_SideBrazed"
+		(property "Footprint" "Package_DIP:DIP-16_W7.62mm"
 			(at 71.12 44.45 0)
 			(effects
@@
 			)
 		)
-		(property "Footprint" "Package_DIP:CERDIP-16_W7.62mm_SideBrazed"
+		(property "Footprint" "Package_DIP:DIP-16_W7.62mm"
 			(at 142.24 99.06 0)
 			(effects
@@
 			)
 		)
-		(property "Footprint" "Capacitor_THT:C_Axial_L3.8mm_D2.6mm_P7.50mm_Horizontal"
+		(property "Footprint" "Capacitor_THT:C_Disc_D3.0mm_W2.0mm_P2.50mm"
 			(at 53.34 59.69 0)
 			(effects
@@
 			)
 		)
-		(property "Footprint" "Package_DIP:CERDIP-16_W7.62mm_SideBrazed"
+		(property "Footprint" "Package_DIP:DIP-16_W7.62mm"
 			(at 130.81 44.45 0)
 			(effects
@@
 			)
 		)
-		(property "Footprint" "Capacitor_THT:C_Axial_L3.8mm_D2.6mm_P7.50mm_Horizontal"
+		(property "Footprint" "Capacitor_THT:C_Disc_D3.0mm_W2.0mm_P2.50mm"
 			(at 113.03 63.5 0)
 			(effects
