File: circuit/Power.kicad_sch (KiCad schematic)
At the start: 17 parts, among them J201 Barrel_Jack, U201 TMA-1215D, U202 LM7805_TO220, U203 LM7905_TO220, U204 LM1117T-3.3

Commit message: Labels for headers on PCB
Parts:
- D201: footprint Diode_THT:D_DO-201AD_P15.24mm_Horizontal -> Diode_THT:D_DO-41_SOD81_P10.16mm_Horizontal
Changed lines of the file:
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@@
 			)
 		)
-		(property "Footprint" "Diode_THT:D_DO-201AD_P15.24mm_Horizontal"
+		(property "Footprint" "Diode_THT:D_DO-41_SOD81_P10.16mm_Horizontal"
 			(at 99.06 47.625 0)
 			(effects
