File: circuit/io_routing.kicad_sch (KiCad schematic)
At the start: 9 parts, among them U101 ADG419BN, U16 CD4051B, U20 CD4051B

Commit message: Created pdf and made minor readabilty changes.
Other:
- title: ESP332 Guitar Patch Bay -> (none)
- moved on the sheet: C113
Changed lines of the file:
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@@
 	(generator "eeschema")
 	(generator_version "9.0")
-	(paper "USLetter")
-	(title_block
-		(title "ESP332 Guitar Patch Bay")
-		(date "2025-05-27")
-		(rev "1")
-	)
+	(paper "A4")
 	(text "Output Mux 1"
 		(exclude_from_sim no)
@@
 	)
 	(junction
-		(at 80.01 96.52)
+		(at 80.01 93.98)
 		(diameter 0)
 		(color 0 0 0 0)
@@
 	)
 	(junction
+		(at 95.25 93.98)
+		(diameter 0)
+		(color 0 0 0 0)
+	)
+	(junction
 		(at 201.93 50.8)
 		(diameter 0)
@@
 	)
 	(junction
-		(at 95.25 96.52)
-		(diameter 0)
-		(color 0 0 0 0)
-	)
-	(junction
 		(at 132.08 142.24)
 		(diameter 0)
@@
 	(wire
 		(pts
-			(xy 95.25 99.06) (xy 95.25 96.52)
+			(xy 95.25 99.06) (xy 95.25 93.98)
 		)
 		(stroke
@@
 	(wire
 		(pts
-			(xy 80.01 96.52) (xy 80.01 106.68)
-		)
-		(stroke
-			(width 0)
-			(type default)
-		)
-	)
-	(wire
-		(pts
 			(xy 186.69 95.25) (xy 189.23 95.25)
 		)
@@
 	(wire
 		(pts
-			(xy 80.01 96.52) (xy 86.36 96.52)
+			(xy 80.01 93.98) (xy 86.36 93.98)
 		)
 		(stroke
@@
 		)
 	)
-	(wire
-		(pts
-			(xy 95.25 90.17) (xy 95.25 96.52)
-		)
-		(stroke
-			(width 0)
-			(type default)
-		)
-	)
 	(bus
 		(pts
@@
 	(wire
 		(pts
+			(xy 95.25 93.98) (xy 95.25 90.17)
+		)
+		(stroke
+			(width 0)
+			(type default)
+		)
+	)
+	(wire
+		(pts
 			(xy 186.69 72.39) (xy 186.69 95.25)
 		)
@@
 		)
 	)
+	(wire
+		(pts
+			(xy 80.01 93.98) (xy 80.01 106.68)
+		)
+		(stroke
+			(width 0)
+			(type default)
+		)
+	)
 	(bus
 		(pts
@@
 	(wire
 		(pts
-			(xy 80.01 72.39) (xy 80.01 96.52)
-		)
-		(stroke
-			(width 0)
-			(type default)
-		)
-	)
-	(wire
-		(pts
 			(xy 199.39 90.17) (xy 199.39 107.95)
 		)
@@
 	(wire
 		(pts
-			(xy 91.44 96.52) (xy 95.25 96.52)
+			(xy 80.01 72.39) (xy 80.01 93.98)
+		)
+		(stroke
+			(width 0)
+			(type default)
+		)
+	)
+	(wire
+		(pts
+			(xy 91.44 93.98) (xy 95.25 93.98)
 		)
 		(stroke
@@
 	(symbol
 		(lib_id "Device:C_Small")
-		(at 88.9 96.52 270)
+		(at 88.9 93.98 270)
 		(unit 1)
 		(exclude_from_sim no)
@@
 		(dnp no)
 		(property "Reference" "C113"
+			(at 88.8936 87.63 90)
+			(effects
+				(font
+					(size 1.27 1.27)
+				)
+			)
+		)
+		(property "Value" "0.1uF"
 			(at 88.8936 90.17 90)
 			(effects
@@
 			)
 		)
-		(property "Value" "0.1uF"
-			(at 88.8936 92.71 90)
-			(effects
-				(font
-					(size 1.27 1.27)
-				)
-			)
-		)
 		(property "Footprint" "Capacitor_THT:C_Axial_L3.8mm_D2.6mm_P7.50mm_Horizontal"
-			(at 88.9 96.52 0)
+			(at 88.9 93.98 0)
 			(effects
 				(font
@@
 		)
 		(property "Datasheet" "~"
-			(at 88.9 96.52 0)
+			(at 88.9 93.98 0)
 			(effects
 				(font
@@
 		)
 		(property "Description" "Unpolarized capacitor, small symbol"
-			(at 88.9 96.52 0)
-			(effects
-				(font
+			(at 88.9 93.98 0)
+			(effects
+				(font

Commit message: Rebuilt Matrix and added inhibit function.
Matrix was flawed, It now supports 8 FX loops (pedals) in any order. Or optionally none at all with a buffered bypass, or anywhere in between. The inhibit function will allow the option to press any loop foot switch an enable or disable it without reprogramming.
Parts:
- removed C113, C114: 0.1uF, Capacitor_THT:C_Axial_L3.8mm_D2.6mm_P7.50mm_Horizontal, symbol Device:C_Small
- removed U16: CD4051B, Package_DIP:CERDIP-16_W7.62mm_SideBrazed, symbol Analog_Switch:CD4051B
Connections:
- net ROW_9 is gone; now on net GUITAR_IN: U101.8
- net U7_Q6 is gone; now on net U7_Q2: U20.10 (B)
- net U7_Q7 is gone; now on net U7_Q3: U20.9 (C)
- net AGND: no longer U20.6 (INH)
- net ROW_1 renamed FX_R_1
- net ROW_2 renamed FX_R_2
- net ROW_3 renamed FX_R_3
- net ROW_4 renamed FX_R_4
- net ROW_5 renamed FX_R_5
- net ROW_6 renamed FX_R_6
- net ROW_7 renamed FX_R_7
- net ROW_8 renamed FX_R_8
- net U7_Q5 renamed U7_Q1
- new net U901_Q0: U20.6 (INH)
Other:
- note removed: "Guitar Routing"

Commit message: Re-annotation of circuit, new PCB routing, updated PDF
Parts:
- renumbered C111 to C401, C112 to C402, C115 to C403, C116 to C404, U101 to U401, U20 to U402
Changed lines of the file:
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@@
 		(on_board yes)
 		(dnp no)
-		(property "Reference" "C111"
+		(property "Reference" "C401"
 			(at 125.73 153.6764 90)
 			(effects
@@
 			(project ""
 				(path "/420e3d7a-6c9a-4806-b4be-05d56aeb21de/eb40e95c-c2ba-417c-afee-eaf028752aed"
-					(reference "C111")
+					(reference "C401")
 					(unit 1)
 				)
@@
 		(dnp no)
 		(fields_autoplaced yes)
-		(property "Reference" "U101"
+		(property "Reference" "U401"
 			(at 143.51 113.03 0)
 			(effects
@@
 			(project ""
 				(path "/420e3d7a-6c9a-4806-b4be-05d56aeb21de/eb40e95c-c2ba-417c-afee-eaf028752aed"
-					(reference "U101")
+					(reference "U401")
 					(unit 1)
 				)
@@
 		(dnp no)
 		(fields_autoplaced yes)
-		(property "Reference" "U101"
+		(property "Reference" "U401"
 			(at 151.13 153.6699 0)
 			(effects
@@
 			(project ""
 				(path "/420e3d7a-6c9a-4806-b4be-05d56aeb21de/eb40e95c-c2ba-417c-afee-eaf028752aed"
-					(reference "U101")
+					(reference "U401")
 					(unit 2)
 				)
@@
 		(on_board yes)
 		(dnp no)
-		(property "Reference" "#PWR0405"
+		(property "Reference" "#PWR0403"
 			(at 222.25 57.15 0)
 			(effects
@@
 			(project "circuit"
 				(path "/420e3d7a-6c9a-4806-b4be-05d56aeb21de/eb40e95c-c2ba-417c-afee-eaf028752aed"
-					(reference "#PWR0405")
+					(reference "#PWR0403")
 					(unit 1)
 				)
@@
 		(on_board yes)
 		(dnp no)
-		(property "Reference" "#PWR0404"
+		(property "Reference" "#PWR0401"
 			(at 143.51 187.96 0)
 			(effects
@@
 			(project "circuit"
 				(path "/420e3d7a-6c9a-4806-b4be-05d56aeb21de/eb40e95c-c2ba-417c-afee-eaf028752aed"
-					(reference "#PWR0404")
+					(reference "#PWR0401")
 					(unit 1)
 				)
@@
 		(on_board yes)
 		(dnp no)
-		(property "Reference" "C115"
+		(property "Reference" "C403"
 			(at 191.7636 88.9 90)
 			(effects
@@
 			(project "circuit"
 				(path "/420e3d7a-6c9a-4806-b4be-05d56aeb21de/eb40e95c-c2ba-417c-afee-eaf028752aed"
-					(reference "C115")
+					(reference "C403")
 					(unit 1)
 				)
@@
 		(on_board yes)
 		(dnp no)
-		(property "Reference" "C116"
+		(property "Reference" "C404"
 			(at 210.8136 44.45 90)
 			(effects
@@
 			(project "circuit"
 				(path "/420e3d7a-6c9a-4806-b4be-05d56aeb21de/eb40e95c-c2ba-417c-afee-eaf028752aed"
-					(reference "C116")
+					(reference "C404")
 					(unit 1)
 				)
@@
 		(dnp no)
 		(fields_autoplaced yes)
-		(property "Reference" "U20"
+		(property "Reference" "U402"
 			(at 204.0733 52.07 0)
 			(effects
@@
 			(project "circuit"
 				(path "/420e3d7a-6c9a-4806-b4be-05d56aeb21de/eb40e95c-c2ba-417c-afee-eaf028752aed"
-					(reference "U20")
+					(reference "U402")
 					(unit 1)
 				)
@@
 		(on_board yes)
 		(dnp no)
-		(property "Reference" "C112"
+		(property "Reference" "C402"
 			(at 158.75 149.8664 90)
 			(effects
@@
 			(project "circuit"
 				(path "/420e3d7a-6c9a-4806-b4be-05d56aeb21de/eb40e95c-c2ba-417c-afee-eaf028752aed"
-					(reference "C112")
-					(unit 1)
-				)
+					(reference "C402")
+					(unit 1)
+				)

Commit message: Added ferrite beads and tweaked PCB
Parts:
- added C405: 0.1uF, Capacitor_THT:C_Disc_D3.0mm_W2.0mm_P2.50mm, symbol Device:C_Small
- C401, C402, C403, C404: footprint Capacitor_THT:C_Axial_L3.8mm_D2.6mm_P7.50mm_Horizontal -> Capacitor_THT:C_Disc_D3.0mm_W2.0mm_P2.50mm
- U402: footprint Package_DIP:CERDIP-16_W7.62mm_SideBrazed -> Package_DIP:DIP-16_W7.62mm
Connections:
- net AGND: now also C405.2
- net +15V renamed +15V_F
- net +5V renamed +5V_F
- net -15V renamed -15V_F
- net -15V_F: now also C405.1
- net -5V renamed -5V_F
Changed lines of the file:
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@@
+	)
+	(junction
+		(at 154.94 167.64)
+		(diameter 0)
+		(color 0 0 0 0)
+	)
+	(junction
+		(at 154.94 173.99)
+		(diameter 0)
+		(color 0 0 0 0)
 	)
 	(junction
@@
 	(wire
 		(pts
-			(xy 165.1 152.4) (xy 165.1 170.18)
+			(xy 165.1 152.4) (xy 165.1 173.99)
 		)
 		(stroke
@@
 		)
 	)
+	(wire
+		(pts
+			(xy 154.94 167.64) (xy 146.05 167.64)
+		)
+		(stroke
+			(width 0)
+			(type default)
+		)
+	)
 	(bus
 		(pts
@@
 	(wire
 		(pts
+			(xy 144.78 173.99) (xy 144.78 170.18)
+		)
+		(stroke
+			(width 0)
+			(type default)
+		)
+	)
+	(wire
+		(pts
 			(xy 196.85 99.06) (xy 196.85 95.25)
 		)
@@
 	(wire
 		(pts
+			(xy 154.94 172.72) (xy 154.94 173.99)
+		)
+		(stroke
+			(width 0)
+			(type default)
+		)
+	)
+	(wire
+		(pts
 			(xy 165.1 147.32) (xy 165.1 139.7)
 		)
@@
 	(wire
 		(pts
-			(xy 158.75 167.64) (xy 146.05 167.64)
+			(xy 144.78 170.18) (xy 143.51 170.18)
+		)
+		(stroke
+			(width 0)
+			(type default)
+		)
+	)
+	(wire
+		(pts
+			(xy 158.75 167.64) (xy 154.94 167.64)
+		)
+		(stroke
+			(width 0)
+			(type default)
+		)
+	)
+	(wire
+		(pts
+			(xy 154.94 173.99) (xy 144.78 173.99)
 		)
 		(stroke
@@
 	(wire
 		(pts
-			(xy 165.1 170.18) (xy 143.51 170.18)
+			(xy 165.1 173.99) (xy 154.94 173.99)
 		)
 		(stroke
@@
 		)
 	)
-	(global_label "+5V"
+	(global_label "+5V_F"
 		(shape input)
 		(at 158.75 137.16 90)
@@
 		)
 	)
-	(global_label "-5V"
+	(global_label "-5V_F"
 		(shape input)
 		(at 196.85 99.06 270)
@@
 		)
 	)
-	(global_label "+5V"
+	(global_label "+5V_F"
 		(shape input)
 		(at 201.93 48.26 90)
@@
 		)
 	)
-	(global_label "+15V"
+	(global_label "+15V_F"
 		(shape input)
 		(at 127 142.24 90)
@@
 		)
 	)
-	(global_label "-15V"
+	(global_label "-15V_F"
 		(shape input)
 		(at 158.75 167.64 90)
@@
 			)
 		)
-		(property "Footprint" "Capacitor_THT:C_Axial_L3.8mm_D2.6mm_P7.50mm_Horizontal"
+		(property "Footprint" "Capacitor_THT:C_Disc_D3.0mm_W2.0mm_P2.50mm"
 			(at 132.08 153.67 0)
 			(effects
@@
 			)
 		)
-		(property "Footprint" "Capacitor_THT:C_Axial_L3.8mm_D2.6mm_P7.50mm_Horizontal"
+		(property "Footprint" "Capacitor_THT:C_Disc_D3.0mm_W2.0mm_P2.50mm"
 			(at 191.77 95.25 0)
 			(effects
@@
 				(path "/420e3d7a-6c9a-4806-b4be-05d56aeb21de/eb40e95c-c2ba-417c-afee-eaf028752aed"
 					(reference "C403")
+					(unit 1)
+				)
+			)
+		)
+	)
+	(symbol
+		(lib_id "Device:C_Small")
+		(at 154.94 170.18 0)
+		(unit 1)
+		(exclude_from_sim no)
+		(in_bom yes)
+		(on_board yes)
+		(dnp no)
+		(property "Reference" "C405"
+			(at 148.59 170.1864 90)
+			(effects
+				(font
+					(size 1.27 1.27)
+				)
+			)
+		)
+		(property "Value" "0.1uF"
+			(at 151.13 170.1864 90)
+			(effects
+				(font
+					(size 1.27 1.27)
+				)
+			)
+		)
+		(property "Footprint" "Capacitor_THT:C_Disc_D3.0mm_W2.0mm_P2.50mm"
+			(at 154.94 170.18 0)
+			(effects
+				(font
+					(size 1.27 1.27)
+				)
+				(hide yes)
+			)
+		)
+		(property "Datasheet" "~"
+			(at 154.94 170.18 0)
+			(effects
+				(font
+					(size 1.27 1.27)
+				)
+				(hide yes)
+			)
+		)
+		(property "Description" "Unpolarized capacitor, small symbol"
+			(at 154.94 170.18 0)
+			(effects
+				(font
+					(size 1.27 1.27)
+				)
+				(hide yes)
+			)
+		)
+		(pin "1"
+		)
+		(pin "2"
+		)
+		(instances
+			(project "circuit"
+				(path "/420e3d7a-6c9a-4806-b4be-05d56aeb21de/eb40e95c-c2ba-417c-afee-eaf028752aed"
+					(reference "C405")
 					(unit 1)
 				)
@@
 			)
 		)
-		(property "Footprint" "Capacitor_THT:C_Axial_L3.8mm_D2.6mm_P7.50mm_Horizontal"
+		(property "Footprint" "Capacitor_THT:C_Disc_D3.0mm_W2.0mm_P2.50mm"
 			(at 210.82 50.8 0)
 			(effects
@@
 			)
 		)
-		(property "Footprint" "Package_DIP:CERDIP-16_W7.62mm_SideBrazed"
+		(property "Footprint" "Package_DIP:DIP-16_W7.62mm"
 			(at 203.2 91.44 0)
 			(effects
@@
 			)
 		)
-		(property "Footprint" "Capacitor_THT:C_Axial_L3.8mm_D2.6mm_P7.50mm_Horizontal"
+		(property "Footprint" "Capacitor_THT:C_Disc_D3.0mm_W2.0mm_P2.50mm"
 			(at 165.1 149.86 0)
 			(effects

Commit message: Circuit tweaks and PCB
Parts:
- C401: footprint Capacitor_THT:C_Disc_D3.0mm_W2.0mm_P2.50mm -> Capacitor_THT:C_Disc_D5.0mm_W2.5mm_P2.50mm
- C402: renamed from C405; footprint Capacitor_THT:C_Disc_D3.0mm_W2.0mm_P2.50mm -> Capacitor_THT:C_Disc_D5.0mm_W2.5mm_P2.50mm
- C403: renamed from C402; footprint Capacitor_THT:C_Disc_D3.0mm_W2.0mm_P2.50mm -> Capacitor_THT:C_Disc_D5.0mm_W2.5mm_P2.50mm
- C404: renamed from C403; footprint Capacitor_THT:C_Disc_D3.0mm_W2.0mm_P2.50mm -> Capacitor_THT:C_Disc_D5.0mm_W2.5mm_P2.50mm
- C405: renamed from C404; footprint Capacitor_THT:C_Disc_D3.0mm_W2.0mm_P2.50mm -> Capacitor_THT:C_Disc_D5.0mm_W2.5mm_P2.50mm
Changed lines of the file:
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@@
 			)
 		)
-		(property "Footprint" "Capacitor_THT:C_Disc_D3.0mm_W2.0mm_P2.50mm"
+		(property "Footprint" "Capacitor_THT:C_Disc_D5.0mm_W2.5mm_P2.50mm"
 			(at 132.08 153.67 0)
 			(effects
@@
 		(on_board yes)
 		(dnp no)
-		(property "Reference" "C403"
+		(property "Reference" "C404"
 			(at 191.7636 88.9 90)
 			(effects
@@
 			)
 		)
-		(property "Footprint" "Capacitor_THT:C_Disc_D3.0mm_W2.0mm_P2.50mm"
+		(property "Footprint" "Capacitor_THT:C_Disc_D5.0mm_W2.5mm_P2.50mm"
 			(at 191.77 95.25 0)
 			(effects
@@
 			(project "circuit"
 				(path "/420e3d7a-6c9a-4806-b4be-05d56aeb21de/eb40e95c-c2ba-417c-afee-eaf028752aed"
-					(reference "C403")
+					(reference "C404")
 					(unit 1)
 				)
@@
 		(on_board yes)
 		(dnp no)
-		(property "Reference" "C405"
+		(property "Reference" "C402"
 			(at 148.59 170.1864 90)
 			(effects
@@
 			)
 		)
-		(property "Footprint" "Capacitor_THT:C_Disc_D3.0mm_W2.0mm_P2.50mm"
+		(property "Footprint" "Capacitor_THT:C_Disc_D5.0mm_W2.5mm_P2.50mm"
 			(at 154.94 170.18 0)
 			(effects
@@
 			(project "circuit"
 				(path "/420e3d7a-6c9a-4806-b4be-05d56aeb21de/eb40e95c-c2ba-417c-afee-eaf028752aed"
-					(reference "C405")
+					(reference "C402")
 					(unit 1)
 				)
@@
 		(on_board yes)
 		(dnp no)
-		(property "Reference" "C404"
+		(property "Reference" "C405"
 			(at 210.8136 44.45 90)
 			(effects
@@
 			)
 		)
-		(property "Footprint" "Capacitor_THT:C_Disc_D3.0mm_W2.0mm_P2.50mm"
+		(property "Footprint" "Capacitor_THT:C_Disc_D5.0mm_W2.5mm_P2.50mm"
 			(at 210.82 50.8 0)
 			(effects
@@
 			(project "circuit"
 				(path "/420e3d7a-6c9a-4806-b4be-05d56aeb21de/eb40e95c-c2ba-417c-afee-eaf028752aed"
-					(reference "C404")
+					(reference "C405")
 					(unit 1)
 				)
@@
 		(on_board yes)
 		(dnp no)
-		(property "Reference" "C402"
+		(property "Reference" "C403"
 			(at 158.75 149.8664 90)
 			(effects
@@
 			)
 		)
-		(property "Footprint" "Capacitor_THT:C_Disc_D3.0mm_W2.0mm_P2.50mm"
+		(property "Footprint" "Capacitor_THT:C_Disc_D5.0mm_W2.5mm_P2.50mm"
 			(at 165.1 149.86 0)
 			(effects
@@
 			(project "circuit"
 				(path "/420e3d7a-6c9a-4806-b4be-05d56aeb21de/eb40e95c-c2ba-417c-afee-eaf028752aed"
-					(reference "C402")
-					(unit 1)
-				)
+					(reference "C403")
+					(unit 1)
+				)

Commit message: Labels for headers on PCB
Connections:
- net U7_Q0 renamed U701_Q0
- net U7_Q1 renamed U701_Q1
- net U7_Q2 renamed U701_Q2
- net U7_Q3 renamed U701_Q3
Changed lines of the file:
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@@
 		)
 	)
-	(label "U7_Q2"
+	(label "U701_Q2"
 		(at 179.07 62.23 0)
 		(effects
@@
 		)
 	)
-	(label "U7_Q0"
+	(label "U701_Q0"
 		(at 132.08 129.54 0)
 		(effects
@@
 		)
 	)
-	(label "U7_Q1"
+	(label "U701_Q1"
 		(at 179.07 59.69 0)
 		(effects
@@
 		)
 	)
-	(label "U7_Q[0..7]"
+	(label "U701_Q[0..7]"
 		(at 55.88 40.64 0)
 		(effects
@@
 		)
 	)
-	(label "U7_Q3"
+	(label "U701_Q3"
 		(at 179.07 64.77 0)
 		(effects
@@
 		)
 	)
-	(hierarchical_label "U7_Q[0..7]"
+	(hierarchical_label "U701_Q[0..7]"
 		(shape output)
 		(at 55.88 43.18 0)
